File: pcb/i2c_led.kicad_pcb (KiCad board)
At the start: 4 copper layers, 20.3 x 14.2 mm, 13 parts, among them J1 Conn_01x05, U1 AW9523B

Commit message: Done with second video https://youtube.com/live/dbczXZmWQ1s?feature=share
Parts:
- added AD0: SolderJumper_3_Bridged12, Jumper:SolderJumper-3_P1.3mm_Bridged2Bar12_RoundedPad1.0x1.5mm, B.Cu at (142.2, 95.2)
- added AD1: SolderJumper_3_Bridged12, Jumper:SolderJumper-3_P1.3mm_Bridged2Bar12_RoundedPad1.0x1.5mm, B.Cu at (142.2, 100.3)
- moved D1 0.25 mm to (153.7, 101.6)
- moved D2 0.25 mm to (153.7, 96.5)
- moved D3 0.25 mm to (153.7, 91.4)
- moved D4 0.25 mm to (148.6, 101.6)
- moved D5 0.25 mm to (148.6, 91.4)
- moved U1 0.13 mm to (149.2, 96.5)
Connections:
- U1 pad 18: VCC -> AD0
- U1 pad 24: VCC -> AD1
Routing:
- net Net-(D3-BK): track 0.00 -> 17.0 mm, vias 0 -> 2
- net VCC: track 9.66 -> 22.9 mm, vias 10 -> 8
- net AD1: track 0.00 -> 8.78 mm, vias 0 -> 1
- net AD0: track 0.00 -> 8.04 mm, vias 0 -> 1
- net Net-(D1-BK): track 0.00 -> 6.60 mm
- net Net-(D2-BK): track 0.00 -> 5.68 mm
- net Net-(D1-GK): track 0.00 -> 5.21 mm
- net Net-(D1-RK): track 0.00 -> 5.13 mm
- net Net-(D4-BK): track 0.00 -> 4.41 mm
- net GND: track 0.00 -> 4.13 mm, vias 0 -> 9
- net Net-(D2-GK): track 0.00 -> 3.69 mm
- net Net-(D4-RK): track 0.00 -> 2.85 mm
- net Net-(D4-GK): track 0.00 -> 2.74 mm
- net Net-(D2-RK): track 0.00 -> 2.36 mm
- net /SCL: track 11.3 -> 13.0 mm
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Other:
- board size 20.3 x 14.2 mm -> 20.3 x 14 mm
- board text added: "${TITLE} rev. ${REVISION}"
- board text added: "GND"
- board text added: "RST"
- board text added: "SCL"
- board text added: "SDA"
- board text added: "VCC"

Commit message: Hmmm
Other:
- board text added: "JLCJLCJLCJLC"
Changed lines of the file:
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@@
 		(title "${TITLE}")
 		(rev "${REVISION}")
+		(company "${COMPANY}")
 		(comment 1 "${AUTHOR}")
 		(comment 2 "${AUTHOR_EMAIL}")
+		(comment 3 "${URL}")
 	)
 	(layers
@@
 			(disableapertmacros no)
 			(usegerberextensions no)
-			(usegerberattributes yes)
+			(usegerberattributes no)
 			(usegerberadvancedattributes yes)
 			(creategerberjobfile yes)
@@
 			(outputformat 1)
 			(mirror no)
-			(drillshape 1)
+			(drillshape 0)
 			(scaleselection 1)
-			(outputdirectory "")
+			(outputdirectory "reva/")
 		)
 	)
 	(property "AUTHOR" "Lars Boegild Thomsen")
 	(property "AUTHOR_EMAIL" "lbthomsen@gmail.com")
+	(property "COMPANY" "STM32World")
 	(property "REVISION" "a")
 	(property "TITLE" "I2C LED")
+	(property "URL" "https://stm32world.com/wiki/I2C_RGB_LED_Board")
 	(net 0 "")
 	(net 1 "GND")
@@
 		(property "Reference" "C1"
 			(at 0 -1.43 90)
+			(unlocked yes)
 			(layer "F.SilkS")
 			(effects
 				(font
-					(size 1 1)
-					(thickness 0.15)
+					(size 0.8 0.8)
+					(thickness 0.1)
 				)
 			)
@@
 		(property "Reference" "R2"
 			(at 0 -1.43 90)
+			(unlocked yes)
 			(layer "F.SilkS")
 			(effects
 				(font
-					(size 1 1)
-					(thickness 0.15)
+					(size 0.8 0.8)
+					(thickness 0.1)
 				)
 			)
@@
 			(effects
 				(font
-					(size 1 1)
+					(size 0.8 0.8)
 					(thickness 0.1)
 				)
@@
 			(effects
 				(font
-					(size 1 1)
+					(size 0.8 0.8)
 					(thickness 0.1)
 				)
@@
 		(property "Reference" "U1"
 			(at 0 -3.33 90)
+			(unlocked yes)
 			(layer "F.SilkS")
 			(effects
 				(font
-					(size 1 1)
-					(thickness 0.15)
+					(size 0.8 0.8)
+					(thickness 0.1)
 				)
 			)
@@
 			)
 		)
+		(property "LCSC" "C965840"
+			(at 0 0 90)
+			(unlocked yes)
+			(layer "F.Fab")
+			(hide yes)
+			(effects
+				(font
+					(size 1 1)
+					(thickness 0.15)
+				)
+			)
+		)
 		(property ki_fp_filters "QFN*1EP*4x4mm*P0.5mm*EP2.7x2.7mm*")
 		(sheetname "/")
@@
 			(effects
 				(font
-					(size 1 1)
+					(size 0.8 0.8)
 					(thickness 0.1)
 				)
@@
 			(effects
 				(font
-					(size 1 1)
+					(size 0.8 0.8)
 					(thickness 0.1)
 				)
@@
 		(property "Reference" "R3"
 			(at 0 -1.43 90)
+			(unlocked yes)
 			(layer "F.SilkS")
 			(effects
 				(font
-					(size 1 1)
-					(thickness 0.15)
+					(size 0.8 0.8)
+					(thickness 0.1)
 				)
 			)
@@
 			(effects
 				(font
-					(size 1 1)
+					(size 0.8 0.8)
 					(thickness 0.1)
 				)
@@
 		(property "Reference" "C3"
 			(at 0 1.27 270)
+			(unlocked yes)
 			(layer "F.SilkS")
 			(effects
 				(font
-					(size 1 1)
-					(thickness 0.15)
+					(size 0.8 0.8)
+					(thickness 0.1)
 				)
 			)
@@
 		(property "Reference" "R1"
 			(at 0 -1.43 90)
+			(unlocked yes)
 			(layer "F.SilkS")
 			(effects
 				(font
-					(size 1 1)
-					(thickness 0.15)
+					(size 0.8 0.8)
+					(thickness 0.1)
 				)
 			)
@@
 		(property "Reference" "J1"
 			(at 0 -2.38 0)
+			(unlocked yes)
 			(layer "F.SilkS")
 			(hide yes)
 			(effects
 				(font
-					(size 1 1)
-					(thickness 0.15)
+					(size 0.8 0.8)
+					(thickness 0.1)
 				)
 			)
@@
 		(sheetname "/")
 		(sheetfile "i2c_led.kicad_sch")
-		(attr through_hole)
+		(attr through_hole exclude_from_bom)
 		(fp_line
 			(start -1.38 -1.38)
@@
 		(property "Reference" "C2"
 			(at 0 -1.43 90)
+			(unlocked yes)
 			(layer "F.SilkS")
 			(effects
 				(font
-					(size 1 1)
-					(thickness 0.15)
+					(size 0.8 0.8)
+					(thickness 0.1)
 				)
 			)
@@
 		(property "Reference" "AD1"
 			(at 0 1.8 0)
+			(unlocked yes)
 			(layer "B.SilkS")
 			(effects
 				(font
-					(size 1 1)
-					(thickness 0.15)
+					(size 0.8 0.8)
+					(thickness 0.1)
 				)
 				(justify mirror)
@@
 		(property "Reference" "AD0"
 			(at 0 1.8 0)
+			(unlocked yes)
 			(layer "B.SilkS")
 			(effects
 				(font
-					(size 1 1)
-					(thickness 0.15)
+					(size 0.8 0.8)
+					(thickness 0.1)
 				)
 				(justify mirror)
@@
 	)
 	(gr_text "${TITLE}\nrev. ${REVISION}"
-		(at 154.94 93.345 0)
+		(at 154.94 90.17 0)
 		(layer "B.SilkS")
 		(effects
 			(font
-				(size 1 1)
+				(size 0.8 0.8)
 				(thickness 0.1)
 			)
-			(justify left bottom mirror)
+			(justify left top mirror)
 		)
 	)
@@
 		(effects
 			(font
-				(size 1 1)
+				(size 0.8 0.8)
 				(thickness 0.1)
 			)
@@
 		(effects
 			(font
-				(size 1 1)
+				(size 0.8 0.8)
 				(thickness 0.1)
 			)
@@
 		(effects
 			(font
-				(size 1 1)
+				(size 0.8 0.8)
 				(thickness 0.1)
 			)
@@
 		)
 	)
+	(gr_text "JLCJLCJLCJLC"
+		(at 154.94 102.87 0)
+		(layer "B.SilkS")
+		(effects
+			(font
+				(size 0.8 0.8)
+				(thickness 0.1)
+			)
+			(justify left bottom mirror)
+		)
+	)
 	(gr_text "SDA"
 		(at 139.7 96.52 90)
@@
 		(effects
 			(font
-				(size 1 1)
+				(size 0.8 0.8)
 				(thickness 0.1)
 			)
@@
 		(effects
 			(font
-				(size 1 1)
+				(size 0.8 0.8)
 				(thickness 0.1)
 			)

Commit message: Tweaked after review
Parts:
- R1, R2: value 1K -> 4k7
- R3: value 100K -> 10k
Changed lines of the file:
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@@
 			)
 		)
-		(property "LCSC" "C1592"
+		(property "LCSC" "C15849"
 			(at 0 0 90)
 			(unlocked yes)
@@
 			)
 		)
-		(property "Value" "1K"
+		(property "Value" "4k7"
 			(at 0 1.43 90)
 			(layer "F.Fab")
@@
 			)
 		)
-		(property "LCSC" "C21190"
+		(property "LCSC" "C23162"
 			(at 0 0 90)
 			(unlocked yes)
@@
 			)
 		)
-		(property "Value" "100K"
+		(property "Value" "10k"
 			(at 0 1.43 90)
 			(layer "F.Fab")
@@
 			)
 		)
-		(property "LCSC" "C14675"
+		(property "LCSC" "C25804"
 			(at 0 0 90)
 			(unlocked yes)
@@
 		(tags "capacitor")
 		(property "Reference" "C3"
-			(at 0 1.27 270)
+			(at 0 1.27 90)
 			(unlocked yes)
 			(layer "F.SilkS")
@@
 			)
 		)
-		(property "Value" "1K"
+		(property "Value" "4k7"
 			(at 0 1.43 90)
 			(layer "F.Fab")
@@
 			)
 		)
-		(property "LCSC" "C21190"
+		(property "LCSC" "C23162"
 			(at 0 0 90)
 			(unlocked yes)

Commit message: Tweaks
Changed lines of the file:
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@@
 	)
 	(via
-		(at 154.305 98.425)
+		(at 154.305 97.79)
 		(size 0.7)
 		(drill 0.35)
@@
 	)
 	(via
-		(at 146.05 90.17)
+		(at 146.05 90.805)
 		(size 0.7)
 		(drill 0.35)
@@
 	)
 	(via
-		(at 146.05 91.44)
+		(at 146.05 92.075)
 		(size 0.7)
 		(drill 0.35)

Commit message: More tweaking
Parts:
- C3: value 100nF -> 1uF
- moved D1 1.27 mm to (154.9, 101.6)
- moved D2 1.27 mm to (154.9, 96.5)
- moved D3 1.27 mm to (154.9, 91.4)
- moved J1 1.27 mm to (135.9, 91.4)
Routing:
- net Net-(D2-BK): track 5.68 -> 8.10 mm
- net Net-(D1-BK): track 6.60 -> 8.19 mm
- net Net-(D2-GK): track 3.69 -> 5.18 mm
- net VCC: track 22.9 -> 24.3 mm
- net Net-(D3-BK): track 17.0 -> 15.6 mm
- net Net-(D2-RK): track 2.36 -> 3.63 mm
- net /SDA: track 10.5 -> 11.7 mm
- net /SCL: track 13.0 -> 14.0 mm
- net Net-(D1-GK): track 5.21 -> 6.18 mm
- net /RSTN: track 13.2 -> 14.0 mm
- net GND: track 4.13 -> 3.43 mm, vias 9 -> 15
- net Net-(D3-GK): track 6.92 -> 7.49 mm
- net Net-(D1-RK): track 5.13 -> 5.68 mm
- net Net-(D4-BK): track 4.41 -> 3.89 mm
Other:
- board size 20.3 x 14 mm -> 22.9 x 14 mm
