File: pcb/i2c_led.kicad_pcb (KiCad board)
At the start: 4 copper layers, 22.9 x 14 mm, 15 parts, among them J1 Conn_01x05, U1 AW9523B

Commit message: More tweaks - should be ready to order
Routing:
- net VCC: vias 8 -> 9
- net GND: vias 15 -> 17
Changed lines of the file:
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@@
 			(keep_text_aligned yes)
 		)
-		(gr_text "550"
+		(gr_text "0.55"
 			(at 130.295 96.52 90)
 			(layer "Dwgs.User")
@@
 			(keep_text_aligned yes)
 		)
-		(gr_text "900"
+		(gr_text "0.9"
 			(at 145.415 86.345 0)
 			(layer "Dwgs.User")
@@
 	)
 	(via
+		(at 139.7 90.805)
+		(size 0.7)
+		(drill 0.35)
+		(layers "F.Cu" "B.Cu")
+		(locked yes)
+		(free yes)
+		(net 1)
+	)
+	(via
 		(at 151.765 90.805)
 		(size 0.7)
@@
 	)
 	(via
-		(at 139.065 102.87)
+		(at 142.875 90.805)
+		(size 0.7)
+		(drill 0.35)
+		(layers "F.Cu" "B.Cu")
+		(free yes)
+		(net 1)
+	)
+	(via
+		(at 139.065 102.235)
 		(size 0.7)
 		(drill 0.35)
@@
 		(drill 0.35)
 		(layers "F.Cu" "B.Cu")
+		(locked yes)
 		(free yes)
 		(net 1)
@@
 	)
 	(segment
-		(start 140.475 92.215)
-		(end 139.7 91.44)
+		(start 137.945 92.215)
+		(end 137.17 91.44)
 		(width 0.3048)
 		(layer "F.Cu")
@@
 	)
 	(segment
-		(start 139.7 91.44)
+		(start 137.17 91.44)
 		(end 135.89 91.44)
 		(width 0.3048)
@@
 	(segment
 		(start 140.97 92.215)
+		(end 142.875 92.215)
+		(width 0.3048)
+		(layer "F.Cu")
+		(net 2)
+	)
+	(segment
+		(start 142.875 92.215)
 		(end 144.145 92.215)
 		(width 0.3048)
@@
 	(segment
 		(start 140.97 92.215)
-		(end 140.475 92.215)
+		(end 137.945 92.215)
 		(width 0.3048)
 		(layer "F.Cu")
@@
 		(size 0.7)
 		(drill 0.35)
+		(layers "F.Cu" "B.Cu")
+		(net 2)
+	)
+	(via
+		(at 142.875 92.215)
+		(size 0.7)
+		(drill 0.35)

Commit message: Ready to order
Other:
- board text added: "${COMPANY}"
Changed lines of the file:
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@@
+		)
+	)
+	(gr_text "${COMPANY}"
+		(at 156.21 101.6 0)
+		(layer "B.SilkS")
+		(effects
+			(font
+				(size 0.8 0.8)
+				(thickness 0.1)
+			)
+			(justify left bottom mirror)
 		)
 	)
@@
 			(keep_text_aligned yes)
 		)
-		(gr_text "0.55"
+		(gr_text "550"
 			(at 130.295 96.52 90)
 			(layer "Dwgs.User")
@@
 			(keep_text_aligned yes)
 		)
-		(gr_text "0.9"
+		(gr_text "900"
 			(at 145.415 86.345 0)
 			(layer "Dwgs.User")
