File: pcb/i2c_led.kicad_pcb (KiCad board)
At the start: 4 copper layers, 22.9 x 14 mm, 15 parts, among them J1 Conn_01x05, U1 AW9523B

Commit message: Added firmware - working
Parts:
- moved AD0 1.27 mm to (142.2, 96.5)
Routing:
- net VCC: track 24.3 -> 23.8 mm
- net GND: vias 17 -> 18
Changed lines of the file:
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@@
 	(property "AUTHOR_EMAIL" "lbthomsen@gmail.com")
 	(property "COMPANY" "STM32World")
-	(property "REVISION" "b")
+	(property "REVISION" "c")
 	(property "TITLE" "I2C LED")
 	(property "URL" "https://stm32world.com/wiki/I2C_RGB_LED_Board")
@@
 	(footprint "Jumper:SolderJumper-3_P1.3mm_Bridged2Bar12_RoundedPad1.0x1.5mm"
 		(layer "B.Cu")
-		(at 142.24 95.25 180)
+		(at 142.24 96.52 180)
 		(descr "SMD Solder 3-pad Jumper, 1x1.5mm rounded Pads, 0.3mm gap, pads 1-2 bridged with 2 copper strip")
 		(tags "net tie solder jumper bridged")
@@
 	)
 	(via
+		(at 146.05 93.345)
+		(size 0.7)
+		(drill 0.35)
+		(layers "F.Cu" "B.Cu")
+		(free yes)
+		(net 1)
+	)
+	(via
 		(at 153.035 95.885)
 		(size 0.7)
@@
 	)
 	(via
-		(at 145.415 94.615)
+		(at 143.51 94.615)
 		(size 0.7)
 		(drill 0.35)
 		(layers "F.Cu" "B.Cu")
+		(locked yes)
 		(free yes)
 		(net 1)
@@
 	)
 	(segment
-		(start 143.54 100.33)
-		(end 143.54 99.03)
-		(width 0.3048)
-		(layer "B.Cu")
-		(net 2)
-	)
-	(segment
 		(start 145.415 96.52)
-		(end 144.145 95.25)
-		(width 0.3048)
+		(end 143.54 96.52)
+		(width 0.2286)
 		(layer "B.Cu")
 		(net 2)
 	)
 	(segment
-		(start 143.54 95.25)
-		(end 144.145 95.25)
+		(start 143.54 100.33)
+		(end 143.54 99.03)
 		(width 0.3048)
 		(layer "B.Cu")
@@
 	)
 	(segment
+		(start 142.6677 93.9973)
+		(end 144.3673 93.9973)
+		(width 0.2286)
+		(layer "F.Cu")
+		(net 20)
+	)
+	(segment
 		(start 139.51 95.695)
 		(end 137.795 93.98)
@@
 	)
 	(segment
-		(start 140.97 94.5)
-		(end 140.97 95.695)
+		(start 147.2625 95.27)
+		(end 145.64 95.27)
 		(width 0.2286)
 		(layer "F.Cu")
@@
 	)
 	(segment
-		(start 141.76 93.71)
-		(end 140.97 94.5)
+		(start 145.3 94.93)
+		(end 145.475 95.105)
 		(width 0.2286)
 		(layer "F.Cu")
@@
 	)
 	(segment
-		(start 145.5 93.71)
-		(end 141.76 93.71)
+		(start 140.97 95.695)
+		(end 142.6677 93.9973)
 		(width 0.2286)
 		(layer "F.Cu")
@@
 	)
 	(segment
-		(start 147.06 95.27)
-		(end 145.5 93.71)
+		(start 145.64 95.27)
+		(end 145.3 94.93)
+		(width 0.2286)
+		(layer "F.Cu")
+		(net 20)
+	)
+	(segment
+		(start 144.3673 93.9973)
+		(end 145.3 94.93)
 		(width 0.2286)
 		(layer "F.Cu")
@@
 	)
 	(segment
-		(start 147.3775 94.5575)
-		(end 147.32 94.615)
+		(start 147.384545 94.5575)
+		(end 147.333502 94.506457)
 		(width 0.2286)
 		(layer "F.Cu")
@@
 	(segment
 		(start 147.975 94.5575)
-		(end 147.3775 94.5575)
+		(end 147.384545 94.5575)
 		(width 0.2286)
 		(layer "F.Cu")
@@
 	)
 	(via
-		(at 147.32 94.615)
+		(at 147.333502 94.506457)
 		(size 0.7)
 		(drill 0.35)
@@
 	)
 	(segment
-		(start 142.24 95.25)
-		(end 142.24 94.2714)
+		(start 142.24 96.52)
+		(end 142.24 95.01144)
+		(width 0.2286)
+		(layer "B.Cu")
+		(net 22)
+	)
+	(segment
+		(start 145.235 94.615)
+		(end 147.224959 94.615)
 		(width 0.2286)
 		(layer "B.Cu")
@@
 	)
 	(segment
-		(start 142.24 94.2714)
-		(end 143.3314 93.18)
+		(start 144.6173 93.9973)
+		(end 145.235 94.615)
 		(width 0.2286)
 		(layer "B.Cu")
@@
 	)
 	(segment
-		(start 147.32 94.17)
-		(end 146.33 93.18)
+		(start 147.224959 94.615)
+		(end 147.333502 94.506457)
 		(width 0.2286)
 		(layer "B.Cu")
@@
 	)
 	(segment
-		(start 147.32 94.615)
-		(end 147.32 94.17)
+		(start 143.25414 93.9973)
+		(end 144.6173 93.9973)
 		(width 0.2286)
 		(layer "B.Cu")
@@
 	)
 	(segment
-		(start 143.3314 93.18)
-		(end 146.33 93.18)
+		(start 142.24 95.01144)
+		(end 143.25414 93.9973)
 		(width 0.2286)
 		(layer "B.Cu")
