File: pcb/i2c_led.kicad_sch (KiCad schematic)
At the start: 13 parts, among them J1 Conn_01x05, U1 AW9523B

Commit message: Done with second video https://youtube.com/live/dbczXZmWQ1s?feature=share
Parts:
- added AD0, AD1: SolderJumper_3_Bridged12, Jumper:SolderJumper-3_P1.3mm_Bridged2Bar12_RoundedPad1.0x1.5mm, symbol Jumper:SolderJumper_3_Bridged12
Connections:
- net GND: now also AD0.3 (B), AD1.3 (B)
- net VCC: now also AD0.1 (A), AD1.1 (A); no longer U1.18 (AD0), U1.24 (AD1)
- new net AD0: AD0.2 (C), U1.18 (AD0)
- new net AD1: AD1.2 (C), U1.24 (AD1)
Other:
- moved on the sheet: C1, C2, C3, D1, D2, D3, D4, D5, J1, R1, R2, R3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

Commit message: Hmmm
Parts:
- J1: now left out of the parts list
- U1: LCSC (none) -> C965840
Changed lines of the file:
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@@
+			)
+		)
+		(property "LCSC" "C965840"
+			(at 151.13 91.44 0)
+			(effects
+				(font
+					(size 1.27 1.27)
+				)
+				(hide yes)
 			)
 		)
@@
 		(unit 1)
 		(exclude_from_sim no)
-		(in_bom yes)
-		(on_board yes)
-		(dnp no)
+		(in_bom no)
+		(on_board yes)
+		(dnp no)

Commit message: Tweaked after review
Parts:
- C1: LCSC C1592 -> C15849
- R1, R2: value 1K -> 4k7; LCSC C21190 -> C23162
- R3: value 100K -> 10k; LCSC C14675 -> C25804
Other:
- moved on the sheet: C1, C2, J1, R1, R2

Commit message: Tweaks
Parts:
- C3: value 100nF -> 1uF; LCSC C14663 -> C15849
Changed lines of the file:
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@@
 			)
 		)
-		(property "Value" "100nF"
+		(property "Value" "1uF"
 			(at 120.396 93.218 0)
 			(effects
@@
 			)
 		)
-		(property "LCSC" "C14663"
+		(property "LCSC" "C15849"
 			(at 119.38 90.17 0)
 			(effects

Commit message: More tweaking
Connections:
- no-connect marks 0 -> 1
Other:
- company: (none) -> ${COMPANY}
- moved on the sheet: AD0, AD1, C1, C2, C3, D1, D2, D3, D4, D5, J1, R1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
